Commit message: joint_state_pub->joint_traj_pub + minor changes

File: iiwa_ros2/iiwa_description/config/iiwa.config.xacro (robot description, xacro)
@@ -1,6 +1,4 @@
 <?xml version="1.0"?>
-<!-- Kuka iiwa 7DoF manipulator -->
 <robot xmlns:xacro="http://www.ros.org/wiki/xacro" name="iiwa">
-    <!-- Enable setting arguments from the launch file -->
     <xacro:arg name="use_sim" default="false" />
     <xacro:arg name="use_fake_hardware" default="true" />
@@ -16,11 +14,7 @@
     <xacro:arg name="namespace" default="/" />
     <xacro:property name="description_package" value="$(arg description_package)"/>
-    <!-- Import iiwa urdf file -->
     <xacro:include filename="$(find ${description_package})/urdf/iiwa.urdf.xacro" />
-    <!-- Import iiwa ros2_control description -->
     <xacro:include filename="$(find ${description_package})/ros2_control/iiwa.r2c_hardware.xacro" />
-    <!-- Import all Gazebo-customization elements -->
     <xacro:include filename="$(find ${description_package})/gazebo/iiwa.gazebo.xacro"/>
-    <!-- Used for fixing robot -->
     <link name="world"/>
     <gazebo reference="world">

File: iiwa_ros2/iiwa_description/gazebo/iiwa.gazebo.xacro (robot description, xacro)
@@ -2,5 +2,4 @@
 <robot xmlns:xacro="http://www.ros.org/wiki/xacro">
   <xacro:macro name="iiwa_gazebo" params="runtime_config_package controllers_file namespace prefix">
-    <!-- ros_control plugin -->
     <gazebo>
       <plugin filename="libgazebo_ros2_control.so" name="gazebo_ros2_control">
@@ -14,5 +13,4 @@
       </plugin>
     </gazebo>
-    <!-- color -->
     <gazebo reference="${prefix}link_7">
       <material>Gazebo/Gray</material>

File: iiwa_ros2/iiwa_description/urdf/iiwa.urdf.xacro (robot description, xacro)
@@ -165,5 +165,5 @@
       <inertial>
         <origin xyz="0 0 0.02" rpy="0 0 0"/>
-        <mass value="${0.3 / 0.308 * 0.44}"/> <!--this is for the MFT Pneumatisch flange-->
+        <mass value="${0.3 / 0.308 * 0.44}"/>
         <inertia ixx="0.01"  ixy="0"  ixz="0" iyy="0.01" iyz="0" izz="0.01" />
       </inertial>
