Commit message: changed to quaternion

File: iiwa_ros2/iiwa_description/urdf/iiwa.urdf.xacro (robot description, xacro)
@@ -12,5 +12,5 @@
   </joint>
   <joint name="${prefix}iiwa_base_joint" type="fixed">
-      <origin rpy="0.0 0 0" xyz="0 0 0"/>
+      <origin rpy="0.0 0 0" xyz="0 0 0.5"/>
       <parent link="${prefix}iiwa_base"/>
       <child link="${prefix}link_0"/>
